File: galgas-didacticas/galgas-didacticas-sch/galgas-didacticas.sch (EAGLE design)
At the start: 0 parts

Commit message: Progress
Parts:
- added C1, C2, C5, C6: 100nF, rcl:C-EUC0805
- added C3, C4: 22pF, rcl:C-EUC0805
- added ICSP: (no value), jumper:JP3Q
- added J1, J2: RJ45_DIRECT, galgas_lib:RJ45_DIRECT
- added JP1: (no value), jumper:JP1E
- added Q1: 16MHz, crystal:CRYSTALHC49UP
- added R1: 120, resistor:R-EU_R0805W
- added U1: ATMEGA328P, atmel:MEGA8-AI
- added U2: MAX481CSA, maxim:MAX481CSA
- added U3: INA128U, burr-brown:INA128U
Connections:
- new net +12V: J1.P3, J2.P3
- new net +5V: U1.VCC@1, U1.VCC@2
- new net /COMMS_RE: U2G$1.RE/
- new net COMMS_A: J1.P2, J2.P2, R1.1, U2G$1.A
- new net COMMS_B: J1.P1, J2.P1, JP1.2, U2G$1.B
- new net COMMS_DE: U2G$1.DE
- new net COMMS_RX: U2G$1.RO
- new net COMMS_TX: U2G$1.DI
- new net GND: C1.2, C2.2, C3.1, C4.2, C5.1, C6.1, J1.GND, J1.P4, J2.GND, J2.P4, U1.GND, U1.GND@1, U1.GND@2
- new net N$1: JP1.1, R1.2
- new net N$2: C6.2, U1.AVCC
- new net N$3: C3.2, Q1.2, U1.PB6(XTAL1/TOSC1)
- new net N$4: C4.1, Q1.1, U1.PB7(XTAL2/TOSC2)
- new net N$5: C5.2, U1.AREF
- new net VCC: C1.1, C2.1
