File: galgas-didacticas/galgas-didacticas-sch/galgas-didacticas.sch (EAGLE design)
At the start: 15 parts, among them J1 RJ45_DIRECT, J2 RJ45_DIRECT, Q1 16MHz, U1 ATMEGA328P, U2 MAX481CSA, U3 INA128U

Commit message: progress
Parts:
- added C10: 1uF, rcl:C-EUC0805
- added C11, C8, C9: 100nF, rcl:C-EUC0805
- added C12: 10uF, rcl:C-EUC0805
- added C13, C14: 10uF, rcl:CPOL-EU153CLV-0505
- added C7: 4.7uF/50V C1206C475K5PACTU, rcl:C-EUC1206K
- added JP3: (no value), jumper:JP2E
- added L1: 6.8uF MLZ2012N6R8LT000, rcl:R-EU_R0805W
- added R2: 100, rcl:R-EU_R0805W
- added R3, R4, R5: 350, resistor:R-EU_R1206W
- added U$1: PEM1-S12-D5-S, galgas_lib:PEM1-S12-D5-S
- added U$2: REF3325, galgas_lib:REF3325
- added U$3: MCP3421, galgas_lib:MCP3421
Connections:
- new net -5V: C14.-, C8.1, U$1.-VO, U3.V-
- new net /RESET: ICSP.3
- new net AGND: C7.2, J1.P4, J2.P4, U$1.GND
- new net G1: U$3.VIN+, U3.OUT
- new net G1N: R3.1, R4.2, U3.-IN
- new net G1P: JP3.2, U3.+IN
- new net MISO: ICSP.1
- new net MOSI: ICSP.5
- new net N$15: JP3.3, R5.2
- new net N$6: L1.2, U$1.VIN
- new net N$7: R2.1, U3.RG
- new net N$8: R2.2, U3.RG@1
- new net SCK: ICSP.2
- new net SCL: U$3.SCL
- new net SDA: U$3.SDA
- new net VREF_2.5V: C10.1, U$2.REF_OUT, U$3.VIN-, U3.REF
- net +12V: now also C7.1, L1.1
- net +5V: now also C11.2, C12.2, C13.+, C9.1, ICSP.6, JP3.1, R3.2, U$1.+VO, U$2.VIN, U$3.VDD, U3.V+
- net GND: now also C10.2, C11.1, C12.1, C13.-, C14.+, C8.2, C9.2, ICSP.4, R4.1, R5.1, U$1.0V, U$2.GND, U$3.VSS; no longer J1.GND, J1.P4, J2.GND, J2.P4
Other:
- moved on the sheet: ICSP, U3

Commit message: First "final" version of the SCH
Parts:
- removed U$1: PEM1-S12-D5-S, galgas_lib:PEM1-S12-D5-S
- removed U$3: MCP3421, galgas_lib:MCP3421
- added LED1, LED2: (no value), jumper:JP1E
- added PT1: 2PT_GND_TIE, SparkFun-Passives:2PT_GND_TIE
- added PWR1: PEM1-S12-D5-S, galgas_lib:PEM1-S12-D5-S
- added Q2, Q3: 2N7002PW, SparkFun-DiscreteSemi:MOSFET-NCHANNEL2N7002PW
- added R6: 10K, resistor:R-EU_R0805W
- added S1: SWITCH-MOMENTARY-2PTH, SparkFun-Electromechanical:SWITCH-MOMENTARY-2PTH
- added U4: MCP3421, galgas_lib:MCP3421
- added U5: REF3325, galgas_lib:REF3325
- U$2: value REF3325 -> SUPPLY_CONNECT; device galgas_lib:REF3325 -> SparkFun-Passives:SUPPLY_CONNECT
Connections:
- new net LED1_PWM: Q2.G, U1.PB1(OC1A)
- new net LED2_PWM: Q3.G, U1.PB2(SS/OC1B)
- new net N$9: LED2.1, Q3.D
- net +12V: now also LED1.2, LED2.2
- net +5V: now also C6.2, ICSP.2, PWR1.+VO, R6.1, U$2.P$1, U1.AVCC, U4.VDD, U5.VIN; no longer ICSP.6, U$1.+VO, U$2.VIN, U$3.VDD
- net -5V: now also PWR1.-VO; no longer U$1.-VO
- net /COMMS_RE: now also U1.PD3(INT1)
- net /RESET: now also ICSP.5, R6.2, S1.2, U1.PC6(/RESET); no longer ICSP.3
- net AGND: now also PT1.P$1, PWR1.GND, Q2.S, Q3.S; no longer U$1.GND
- net COMMS_DE: now also U1.PD2(INT0)
- net COMMS_RX: now also U1.PD0(RXD)
- net COMMS_TX: now also U1.PD1(TXD)
- net G1: now also U4.VIN+; no longer U$3.VIN+
- net GND: now also ICSP.6, PT1.P$2, PWR1.0V, S1.1, U4.VSS, U5.GND; no longer ICSP.4, U$1.0V, U$2.GND, U$3.VSS
- net MISO: now also U1.PB4(MISO)
- net MOSI: now also ICSP.4, U1.PB3(MOSI/OC2); no longer ICSP.5
- net N$2: now also LED1.1, Q2.D; no longer C6.2, U1.AVCC
- net N$6: now also PWR1.VIN; no longer U$1.VIN
- net SCK: now also ICSP.3, U1.PB5(SCK); no longer ICSP.2
- net SCL: now also U1.PC5(ADC5/SCL), U4.SCL; no longer U$3.SCL
- net SDA: now also U1.PC4(ADC4/SDA), U4.SDA; no longer U$3.SDA
- net VCC: now also U$2.P$2
- net VREF_2.5V: now also U4.VIN-, U5.REF_OUT; no longer U$2.REF_OUT, U$3.VIN-
Other:
- note added: "LEDS"
- note added: "Módulo: Galgas + tiras LED PWM"
- note added: "Parte analógica"
- note added: "Power"
- note added: "RJ45"
- note added: "RS422 comms."
- note added: "uC"
- moved on the sheet: C1, C10, C11, C12, C13, C14, C2, C3, C4, C5, C6, C7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

Commit message: Board routing done
Parts:
- Q1: value 16MHz -> 16M
Connections:
- net +12V: now also J1.P8, J2.P8; no longer J1.P3, J2.P3
- net +5V: now also C2.1
- net AGND: now also J1.P6, J2.P6; no longer J1.P4, J2.P4
- net VCC: no longer C2.1
Other:
- moved on the sheet: C1
Changed lines of the file:
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@@
 <part name="GND7" library="supply1" deviceset="GND" device=""/>
 <part name="P+6" library="supply1" deviceset="+5V" device=""/>
-<part name="Q1" library="crystal" deviceset="CRYSTAL" device="HC49UP" value="16MHz"/>
+<part name="Q1" library="crystal" deviceset="CRYSTAL" device="HC49UP" value="16M"/>
 <part name="C2" library="rcl" deviceset="C-EU" device="C0805" value="100nF"/>
-<part name="P+7" library="supply1" deviceset="VCC" device=""/>
 <part name="GND8" library="supply1" deviceset="GND" device=""/>
 <part name="C3" library="rcl" deviceset="C-EU" device="C0805" value="22pF"/>
@@
 <part name="P+17" library="supply1" deviceset="VCC" device=""/>
 <part name="P+18" library="supply1" deviceset="+5V" device=""/>
+<part name="P+7" library="supply1" deviceset="+5V" device=""/>
 </parts>
 <sheets>
@@
 <instance part="J1" gate="G$1" x="-60.96" y="58.42" rot="R180"/>
 <instance part="J2" gate="G$1" x="-60.96" y="25.4" rot="R180"/>
-<instance part="P+1" gate="1" x="-99.06" y="58.42"/>
-<instance part="P+2" gate="1" x="-96.52" y="25.4"/>
+<instance part="P+1" gate="1" x="-83.82" y="63.5" rot="R90"/>
+<instance part="P+2" gate="1" x="-91.44" y="30.48" rot="R90"/>
 <instance part="U2" gate="G$1" x="-162.56" y="53.34" rot="MR180"/>
 <instance part="R1" gate="G$1" x="-139.7" y="30.48" rot="R90"/>
 <instance part="JP1" gate="A" x="-142.24" y="38.1" rot="R90"/>
-<instance part="C1" gate="G$1" x="-124.46" y="-5.08"/>
-<instance part="P+5" gate="VCC" x="-124.46" y="0"/>
-<instance part="GND5" gate="1" x="-124.46" y="-12.7"/>
+<instance part="C1" gate="G$1" x="-198.12" y="35.56"/>
+<instance part="P+5" gate="VCC" x="-198.12" y="40.64"/>
+<instance part="GND5" gate="1" x="-198.12" y="27.94"/>
 <instance part="U3" gate="G$1" x="-261.62" y="121.92"/>
 <instance part="U1" gate="G$1" x="-312.42" y="12.7"/>
@@
 <instance part="Q1" gate="G$1" x="-355.6" y="17.78" rot="R90"/>
 <instance part="C2" gate="G$1" x="-358.14" y="-12.7"/>
-<instance part="P+7" gate="VCC" x="-358.14" y="-7.62"/>
 <instance part="GND8" gate="1" x="-358.14" y="-20.32"/>
 <instance part="C3" gate="G$1" x="-368.3" y="20.32" rot="R90"/>
@@
 <instance part="GND13" gate="1" x="-373.38" y="50.8" rot="R180"/>
 <instance part="P+8" gate="1" x="-226.06" y="-22.86" rot="R90"/>
-<instance part="AGND1" gate="VR1" x="-78.74" y="53.34" rot="R270"/>
-<instance part="AGND2" gate="VR1" x="-78.74" y="20.32" rot="R270"/>
+<instance part="AGND1" gate="VR1" x="-73.66" y="58.42" rot="R270"/>
+<instance part="AGND2" gate="VR1" x="-78.74" y="25.4" rot="R270"/>
 <instance part="AGND3" gate="VR1" x="-213.36" y="-45.72"/>
 <instance part="GND1" gate="1" x="-142.24" y="-33.02" rot="R90"/>
@@
 <instance part="P+17" gate="VCC" x="-170.18" y="-5.08" rot="R270"/>
 <instance part="P+18" gate="1" x="-190.5" y="-5.08" rot="R90"/>
+<instance part="P+7" gate="1" x="-358.14" y="-7.62"/>
 </instances>
 <busses>
@@
 <net name="+12V" class="0">
 <segment>
-<pinref part="J1" gate="G$1" pin="P3"/>
-<pinref part="P+1" gate="1" pin="+12V"/>
-<wire x1="-68.58" y1="50.8" x2="-99.06" y2="50.8" width="0.1524" layer="91"/>
-<wire x1="-99.06" y1="50.8" x2="-99.06" y2="55.88" width="0.1524" layer="91"/>
-</segment>
-<segment>
-<pinref part="J2" gate="G$1" pin="P3"/>
-<pinref part="P+2" gate="1" pin="+12V"/>
-<wire x1="-68.58" y1="17.78" x2="-96.52" y2="17.78" width="0.1524" layer="91"/>
-<wire x1="-96.52" y1="17.78" x2="-96.52" y2="22.86" width="0.1524" layer="91"/>
-</segment>
-<segment>
 <pinref part="P+8" gate="1" pin="+12V"/>
 <pinref part="C7" gate="G$1" pin="1"/>
@@
 <wire x1="-43.18" y1="-17.78" x2="-43.18" y2="-12.7" width="0.1524" layer="91"/>
 </segment>
+<segment>
+<pinref part="P+1" gate="1" pin="+12V"/>
+<pinref part="J1" gate="G$1" pin="P8"/>
+<wire x1="-81.28" y1="63.5" x2="-68.58" y2="63.5" width="0.1524" layer="91"/>
+</segment>
+<segment>
+<pinref part="P+2" gate="1" pin="+12V"/>
+<pinref part="J2" gate="G$1" pin="P8"/>
+<wire x1="-88.9" y1="30.48" x2="-68.58" y2="30.48" width="0.1524" layer="91"/>
+</segment>
 </net>
 <net name="VCC" class="0">
@@
 <pinref part="C1" gate="G$1" pin="1"/>
 <pinref part="P+5" gate="VCC" pin="VCC"/>
-</segment>
-<segment>
-<pinref part="C2" gate="G$1" pin="1"/>
-<pinref part="P+7" gate="VCC" pin="VCC"/>
 </segment>
 <segment>
@@
 <pinref part="P+18" gate="1" pin="+5V"/>
 </segment>
+<segment>
+<pinref part="C2" gate="G$1" pin="1"/>
+<pinref part="P+7" gate="1" pin="+5V"/>
+</segment>
 </net>
 <net name="N$3" class="0">
@@
 <net name="AGND" class="0">
 <segment>
-<pinref part="J1" gate="G$1" pin="P4"/>
-<wire x1="-76.2" y1="53.34" x2="-68.58" y2="53.34" width="0.1524" layer="91"/>
-<pinref part="AGND1" gate="VR1" pin="AGND"/>
-</segment>
-<segment>
-<pinref part="J2" gate="G$1" pin="P4"/>
-<wire x1="-76.2" y1="20.32" x2="-68.58" y2="20.32" width="0.1524" layer="91"/>
-<pinref part="AGND2" gate="VR1" pin="AGND"/>
-</segment>
-<segment>
 <pinref part="AGND3" gate="VR1" pin="AGND"/>
 <wire x1="-213.36" y1="-43.18" x2="-182.88" y2="-43.18" width="0.1524" layer="91"/>
@@
 <pinref part="AGND6" gate="VR1" pin="AGND"/>
 </segment>
-</net>
+<segment>
+<pinref part="AGND1" gate="VR1" pin="AGND"/>
+<pinref part="J1" gate="G$1" pin="P6"/>
+<wire x1="-71.12" y1="58.42" x2="-68.58" y2="58.42" width="0.1524" layer="91"/>
+</segment>
+<segment>
+<pinref part="AGND2" gate="VR1" pin="AGND"/>
+<pinref part="J2" gate="G$1" pin="P6"/>
+<wire x1="-76.2" y1="25.4" x2="-68.58" y2="25.4" width="0.1524" layer="91"/>
+</segment>
+</net>

Commit message: mejoras (más condensadores desacoplo, etc.)
Parts:
- added C15: 100uF, rcl:CPOL-EU153CLV-0505
- added C16, C17, C18: 100nF, rcl:C-EUC0805
- added R7, R8: 3.3K, resistor:R-EU_R0805W
Connections:
- net +5V: now also C15.+, C16.1, C17.1, R7.1, R8.1
- net GND: now also C15.-, C16.2, C17.2, C18.1
- net SCL: now also R8.2
- net SDA: now also R7.2
- net VREF_2.5V: now also C18.2
Changed lines of the file:
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@@
 <part name="P+18" library="supply1" deviceset="+5V" device=""/>
 <part name="P+7" library="supply1" deviceset="+5V" device=""/>
+<part name="C15" library="rcl" deviceset="CPOL-EU" device="153CLV-0505" value="100uF"/>
+<part name="C16" library="rcl" deviceset="C-EU" device="C0805" value="100nF"/>
+<part name="GND23" library="supply1" deviceset="GND" device=""/>
+<part name="GND24" library="supply1" deviceset="GND" device=""/>
+<part name="C17" library="rcl" deviceset="C-EU" device="C0805" value="100nF"/>
+<part name="GND25" library="supply1" deviceset="GND" device=""/>
+<part name="P+19" library="supply1" deviceset="+5V" device=""/>
+<part name="P+20" library="supply1" deviceset="+5V" device=""/>
+<part name="R7" library="resistor" deviceset="R-EU_" device="R0805W" value="3.3K"/>
+<part name="R8" library="resistor" deviceset="R-EU_" device="R0805W" value="3.3K"/>
+<part name="C18" library="rcl" deviceset="C-EU" device="C0805" value="100nF"/>
+<part name="GND26" library="supply1" deviceset="GND" device=""/>
 </parts>
 <sheets>
@@
 <instance part="C9" gate="G$1" x="-220.98" y="104.14"/>
 <instance part="GND3" gate="1" x="-220.98" y="96.52"/>
-<instance part="P+11" gate="1" x="-109.22" y="116.84" rot="R90"/>
+<instance part="P+11" gate="1" x="-119.38" y="116.84" rot="R90"/>
 <instance part="GND4" gate="1" x="-86.36" y="101.6"/>
 <instance part="C10" gate="G$1" x="-58.42" y="114.3"/>
@@
 <instance part="GND17" gate="1" x="-144.78" y="124.46" rot="R180"/>
 <instance part="GND18" gate="1" x="-340.36" y="91.44"/>
-<instance part="P+13" gate="1" x="-340.36" y="152.4"/>
+<instance part="P+13" gate="1" x="-340.36" y="157.48"/>
 <instance part="C13" gate="G$1" x="-132.08" y="-25.4"/>
 <instance part="C14" gate="G$1" x="-132.08" y="-48.26" rot="R180"/>
@@
 <instance part="P+18" gate="1" x="-190.5" y="-5.08" rot="R90"/>
 <instance part="P+7" gate="1" x="-358.14" y="-7.62"/>
+<instance part="C15" gate="G$1" x="-327.66" y="149.86"/>
+<instance part="C16" gate="G$1" x="-317.5" y="149.86"/>
+<instance part="GND23" gate="1" x="-327.66" y="142.24"/>
+<instance part="GND24" gate="1" x="-317.5" y="142.24"/>
+<instance part="C17" gate="G$1" x="-111.76" y="106.68"/>
+<instance part="GND25" gate="1" x="-111.76" y="99.06"/>
+<instance part="P+19" gate="1" x="-266.7" y="45.72"/>
+<instance part="P+20" gate="1" x="-256.54" y="45.72"/>
+<instance part="R7" gate="G$1" x="-266.7" y="35.56" rot="R270"/>
+<instance part="R8" gate="G$1" x="-256.54" y="35.56" rot="R270"/>
+<instance part="C18" gate="G$1" x="-233.68" y="127"/>
+<instance part="GND26" gate="1" x="-233.68" y="132.08" rot="R180"/>
 </instances>
 <busses>
@@
 <pinref part="GND6" gate="1" pin="GND"/>
 </segment>
+<segment>
+<pinref part="C15" gate="G$1" pin="-"/>
+<pinref part="GND23" gate="1" pin="GND"/>
+</segment>
+<segment>
+<pinref part="C16" gate="G$1" pin="2"/>
+<pinref part="GND24" gate="1" pin="GND"/>
+</segment>
+<segment>
+<pinref part="C17" gate="G$1" pin="2"/>
+<pinref part="GND25" gate="1" pin="GND"/>
+</segment>
+<segment>
+<pinref part="C18" gate="G$1" pin="1"/>
+<pinref part="GND26" gate="1" pin="GND"/>
+</segment>
 </net>
 <net name="COMMS_B" class="0">
@@
 </segment>
 <segment>
-<wire x1="-340.36" y1="149.86" x2="-340.36" y2="137.16" width="0.1524" layer="91"/>
+<wire x1="-340.36" y1="154.94" x2="-340.36" y2="152.4" width="0.1524" layer="91"/>
 <pinref part="R3" gate="G$1" pin="2"/>
+<wire x1="-340.36" y1="152.4" x2="-340.36" y2="137.16" width="0.1524" layer="91"/>
 <wire x1="-355.6" y1="127" x2="-355.6" y2="137.16" width="0.1524" layer="91"/>
 <wire x1="-355.6" y1="137.16" x2="-340.36" y2="137.16" width="0.1524" layer="91"/>
@@
 <pinref part="P+13" gate="1" pin="+5V"/>
 <junction x="-340.36" y="137.16"/>
+<pinref part="C16" gate="G$1" pin="1"/>
+<pinref part="C15" gate="G$1" pin="+"/>
+<wire x1="-317.5" y1="152.4" x2="-327.66" y2="152.4" width="0.1524" layer="91"/>
+<wire x1="-327.66" y1="152.4" x2="-340.36" y2="152.4" width="0.1524" layer="91"/>
+<junction x="-327.66" y="152.4"/>
+<junction x="-340.36" y="152.4"/>
 </segment>
 <segment>
@@
 <pinref part="P+11" gate="1" pin="+5V"/>
 <pinref part="U5" gate="G$1" pin="VIN"/>
+<wire x1="-116.84" y1="116.84" x2="-111.76" y2="116.84" width="0.1524" layer="91"/>
+<pinref part="C17" gate="G$1" pin="1"/>
+<wire x1="-111.76" y1="116.84" x2="-106.68" y2="116.84" width="0.1524" layer="91"/>
+<wire x1="-111.76" y1="109.22" x2="-111.76" y2="116.84" width="0.1524" layer="91"/>
+<junction x="-111.76" y="116.84"/>
 </segment>
 <segment>
@@
 <pinref part="C2" gate="G$1" pin="1"/>
 <pinref part="P+7" gate="1" pin="+5V"/>
+</segment>
+<segment>
+<pinref part="R7" gate="G$1" pin="1"/>
+<pinref part="P+19" gate="1" pin="+5V"/>
+<wire x1="-266.7" y1="40.64" x2="-266.7" y2="43.18" width="0.1524" layer="91"/>
+</segment>
+<segment>
+<pinref part="R8" gate="G$1" pin="1"/>
+<pinref part="P+20" gate="1" pin="+5V"/>
+<wire x1="-256.54" y1="40.64" x2="-256.54" y2="43.18" width="0.1524" layer="91"/>
 </segment>
 </net>
@@
 <segment>
 <pinref part="U3" gate="G$1" pin="REF"/>
-<wire x1="-243.84" y1="116.84" x2="-231.14" y2="116.84" width="0.1524" layer="91"/>
+<wire x1="-243.84" y1="116.84" x2="-233.68" y2="116.84" width="0.1524" layer="91"/>
 <label x="-231.14" y="116.84" size="1.778" layer="95"/>
+<pinref part="C18" gate="G$1" pin="2"/>
+<wire x1="-233.68" y1="116.84" x2="-231.14" y2="116.84" width="0.1524" layer="91"/>
+<wire x1="-233.68" y1="121.92" x2="-233.68" y2="116.84" width="0.1524" layer="91"/>
+<junction x="-233.68" y="116.84"/>
 </segment>
 <segment>
@@
 <segment>
 <pinref part="U3" gate="G$1" pin="OUT"/>
-<wire x1="-243.84" y1="124.46" x2="-226.06" y2="124.46" width="0.1524" layer="91"/>
-<label x="-228.6" y="124.46" size="1.778" layer="95"/>
+<wire x1="-243.84" y1="124.46" x2="-238.76" y2="124.46" width="0.1524" layer="91"/>
+<label x="-241.3" y="124.46" size="1.778" layer="95"/>
 </segment>
 <segment>
@@
 <segment>
 <pinref part="U1" gate="G$1" pin="PC5(ADC5/SCL)"/>
-<wire x1="-287.02" y1="25.4" x2="-276.86" y2="25.4" width="0.1524" layer="91"/>
 <label x="-279.4" y="25.4" size="1.778" layer="95"/>
+<pinref part="R8" gate="G$1" pin="2"/>
+<wire x1="-287.02" y1="25.4" x2="-256.54" y2="25.4" width="0.1524" layer="91"/>
+<wire x1="-256.54" y1="25.4" x2="-256.54" y2="30.48" width="0.1524" layer="91"/>
 </segment>
 </net>
@@
 <segment>
 <pinref part="U1" gate="G$1" pin="PC4(ADC4/SDA)"/>
-<wire x1="-287.02" y1="27.94" x2="-276.86" y2="27.94" width="0.1524" layer="91"/>
 <label x="-279.4" y="27.94" size="1.778" layer="95"/>
+<pinref part="R7" gate="G$1" pin="2"/>
+<wire x1="-287.02" y1="27.94" x2="-266.7" y2="27.94" width="0.1524" layer="91"/>
+<wire x1="-266.7" y1="27.94" x2="-266.7" y2="30.48" width="0.1524" layer="91"/>
 </segment>
 </net>
@@
 </sheet>
 </sheets>
+<errors>
+</errors>
 </schematic>
 </drawing>
